Commit message: fix(pipeline): Bug 28。根元リンクの原点を第1関節の XY にする
glb_to_links が根元リンクのローカル原点を XY=(0,0) 決め打ちにしていた。
GLB の原点が台座の真下にあるとは限らず、A1 では台座が x∈[-0.332,-0.157] に
あって原点が形状の 0.157 m 外に出ていた。URDF の world_to_base は Z 軸まわりの
回転なので、台座が自分から 0.16〜0.33 m 離れた軸のまわりを公転していた。

Bug 27 と同じ構図で、「GLB は原点中心に鉛直な腕が立っている」という暗黙の前提を
A1 が初めて破った。v2c では J1 の XY がたまたま原点と一致していた
（A1 の J1 は (-0.2428,-0.0094)、v2c は (+0.0004,-0.0002)）。

影響は可視化のみ。学習用 XML は台座メッシュを使わず body "0" は球で、
FIXED_BASE=1 により台座は topology.json に入らない。修正前後で topology.json が
バイト単位で変化しないことを確認したので、稼働中の学習に手は入れていない。

修正後は台座 STL が x∈[-0.089,+0.085] となり原点が内側に入った。URDF の
joint_to_upper_arm の原点も (0,0,0.2195) になり第1関節が台座の真上に来る。
副次的に台座の link_length（台座高）も 0.3276 → 0.2195 m と正しくなった。

Co-Authored-By: Claude Opus 5 <noreply@anthropic.com>

File: data/test/A1/e2e_a1.urdf (robot description, URDF)
Before this commit: robot tripo_arm, 5 links, 4 joints
Joints:
- joint joint_to_upper_arm: origin xyz=-0.242760 -0.009414 0.219532 rpy=0 0 0 -> xyz=0.000000 0.000000 0.219532 rpy=0 0 0
